Commit message: gui and non gui launch files, added changable JSP

File: src/scara_kinematics/urdf/arm.urdf (robot description, URDF)
Before this commit: robot test arm, 1 links, 0 joints
Links:
- added link base_extension; visual box size=1 .1 .1
- added link dummy_rotation_link
- added link end_link; visual box size=.1 .1 1
- added link middle_link; visual box size=1 .1 .1
- link base_link: geometry visual cylinder length=2 radius=0.1
Joints:
- added joint d_3: type prismatic, parent dummy_rotation_link, child end_link, origin xyz=1.05 0 0, axis 0 0 1, limit lower=-0.5 upper=0.5 effort=30 velocity=1.0
- added joint dummy_rotation: type revolute, parent middle_link, child dummy_rotation_link, origin xyz=0 0 0, axis 1 0 0, limit lower=3.14159 upper=3.14159 effort=30 velocity=1.0
- added joint theta_1: type continuous, parent base_link, child base_extension, origin xyz=0 0 2, axis 0 0 1
- added joint theta_2: type continuous, parent base_extension, child middle_link, origin xyz=1 0 0, axis 0 0 1

Commit message: gazebo development, no model visible

File: src/scara_kinematics/urdf/arm.urdf (robot description, URDF)
Before this commit: robot test arm, 5 links, 4 joints
Links:
- link base_extension: mass None -> 1
- link base_link: mass None -> 1
- link dummy_rotation_link: mass None -> 1
- link end_link: mass None -> 1
- link middle_link: mass None -> 1
Joints:
- joint dummy_rotation: limit lower=3.14159 upper=3.14159 effort=30 velocity=1.0 -> lower=3.14 upper=3.15 effort=30 velocity=1.0
