Commit message: assignment2-partialy-working

File: src/scara_kinematics/urdf/arm_gazebo.urdf (robot description, URDF)
Before this commit: robot test_arm, 6 links, 5 joints
Links:
- link end_link: mass .01 -> 1
Joints:
- joint theta_1: type revolute -> fixed
- joint theta_2: type continuous -> fixed

Commit message: working

File: src/scara_kinematics/urdf/arm_gazebo.urdf (robot description, URDF)
Before this commit: robot test_arm, 6 links, 5 joints
Links:
- link end_link: mass 1 -> .1; geometry visual box size=.1 .1 2
Joints:
- joint d_3: limit lower=-0.5 upper=0.5 effort=100 velocity=.3 -> lower=-1 upper=1 effort=100 velocity=.3; origin xyz=1.0 0 0.5 -> xyz=1.0 0 1
- joint theta_1: limit lower=-1.6 upper=1.6 effort=100 velocity=0.3 -> lower=-3.14159 upper=3.13159 effort=100 velocity=0.3; type fixed -> revolute
- joint theta_2: limit lower=-1.6 upper=1.6 effort=100 velocity=0.3 -> lower=-3.14159 upper=3.14159 effort=100 velocity=0.3; type fixed -> revolute
